Commit message: 6 dof continuous movement

File: src/space_printer_description/urdf/space_printer.urdf (robot description, URDF)
Before this commit: robot space_printer_bot, 8 links, 7 joints
Links:
- link extruder_nozzle: geometry visual cylinder length=0.1 radius=0.05

Commit message: gazebo is added instead of rezviz

File: src/space_printer_description/urdf/space_printer.urdf (robot description, URDF)
Before this commit: robot space_printer_bot, 8 links, 7 joints
Links:
- added link world
- link base_link: mass None -> 1.0
- link extruder_nozzle: mass None -> 1.0
- link link_1: mass None -> 1.0
- link link_2: mass None -> 1.0
- link link_3: mass None -> 1.0
- link link_4: mass None -> 1.0
- link link_5: mass None -> 1.0
- link link_6: mass None -> 1.0
Joints:
- added joint fixed_to_world: type fixed, parent world, child base_link
