Commit message: wheel of turtlebot3 is speening although size of the 6 dof needs to be smaller

File: install/space_printer_description/share/space_printer_description/urdf/space_printer.urdf (robot description, URDF)
Before this commit: robot space_printer_bot, 8 links, 7 joints
Links:
- removed link base_link
- added link arm_base_link, mass 1.0; visual cylinder length=0.1 radius=0.1
- link extruder_nozzle: mass None -> 1.0; geometry visual cylinder length=0.1 radius=0.05
- link link_1: mass None -> 1.0
- link link_2: mass None -> 1.0
- link link_3: mass None -> 1.0
- link link_4: mass None -> 1.0
- link link_5: mass None -> 1.0
- link link_6: mass None -> 1.0
Joints:
- joint joint_1: parent base_link -> arm_base_link

File: src/space_printer_description/urdf/space_printer.urdf (robot description, URDF)
Before this commit: robot space_printer_bot, 9 links, 8 joints
Links:
- removed link base_link
- removed link world
- added link arm_base_link, mass 1.0; visual cylinder length=0.1 radius=0.1
Joints:
- removed joint fixed_to_world
- joint joint_1: parent base_link -> arm_base_link

Commit message: matlab command is added

File: install/space_printer_description/share/space_printer_description/urdf/space_printer.urdf (robot description, URDF)
Before this commit: robot space_printer_bot, 8 links, 7 joints
Links:
- link arm_base_link: mass 1.0 -> 5; geometry visual cylinder length=0.05 radius=0.05
- link extruder_nozzle: mass 1.0 -> 0.05; geometry visual cylinder length=0.05 radius=0.025
- link link_1: mass 1.0 -> 0.05; geometry visual cylinder length=0.1 radius=0.04
- link link_2: mass 1.0 -> 0.05; geometry visual cylinder length=0.2 radius=0.03
- link link_3: mass 1.0 -> 0.05; geometry visual cylinder length=0.15 radius=0.025
- link link_4: mass 1.0 -> 0.05; geometry visual cylinder length=0.05 radius=0.02
- link link_5: mass 1.0 -> 0.05; geometry visual cylinder length=0.05 radius=0.02
- link link_6: mass 1.0 -> 0.05; geometry visual cylinder length=0.025 radius=0.02
Joints:
- joint extruder_joint: origin xyz=0 0 0.05 rpy=0 0 0 -> xyz=0 0 0.025 rpy=0 0 0
- joint joint_1: origin xyz=0 0 0.05 rpy=0 0 0 -> xyz=0 0 0.025 rpy=0 0 0
- joint joint_2: origin xyz=0 0 0.2 rpy=0 0 0 -> xyz=0 0 0.1 rpy=0 0 0
- joint joint_3: origin xyz=0 0 0.4 rpy=0 0 0 -> xyz=0 0 0.2 rpy=0 0 0
- joint joint_4: origin xyz=0 0 0.3 rpy=0 0 0 -> xyz=0 0 0.15 rpy=0 0 0
- joint joint_5: origin xyz=0 0 0.1 rpy=0 0 0 -> xyz=0 0 0.05 rpy=0 0 0
- joint joint_6: origin xyz=0 0 0.1 rpy=0 0 0 -> xyz=0 0 0.05 rpy=0 0 0

File: src/space_printer_description/urdf/turtlebot_miner.urdf (robot description, URDF)
Before this commit: robot turtlebot_miner, 21 links, 20 joints
Links:
- link arm_base_link: mass 1.0 -> 5; geometry visual cylinder length=0.05 radius=0.05
- link extruder_nozzle: mass 1.0 -> 0.05; geometry visual cylinder length=0.05 radius=0.025
- link link_1: mass 1.0 -> 0.05; geometry visual cylinder length=0.1 radius=0.04
- link link_2: mass 1.0 -> 0.05; geometry visual cylinder length=0.2 radius=0.03
- link link_3: mass 1.0 -> 0.05; geometry visual cylinder length=0.15 radius=0.025
- link link_4: mass 1.0 -> 0.05; geometry visual cylinder length=0.05 radius=0.02
- link link_5: mass 1.0 -> 0.05; geometry visual cylinder length=0.05 radius=0.02
- link link_6: mass 1.0 -> 0.05; geometry visual cylinder length=0.025 radius=0.02
Joints:
- joint extruder_joint: origin xyz=0 0 0.05 rpy=0 0 0 -> xyz=0 0 0.025 rpy=0 0 0
- joint joint_1: origin xyz=0 0 0.05 rpy=0 0 0 -> xyz=0 0 0.025 rpy=0 0 0
- joint joint_2: origin xyz=0 0 0.2 rpy=0 0 0 -> xyz=0 0 0.1 rpy=0 0 0
- joint joint_3: origin xyz=0 0 0.4 rpy=0 0 0 -> xyz=0 0 0.2 rpy=0 0 0
- joint joint_4: origin xyz=0 0 0.3 rpy=0 0 0 -> xyz=0 0 0.15 rpy=0 0 0
- joint joint_5: origin xyz=0 0 0.1 rpy=0 0 0 -> xyz=0 0 0.05 rpy=0 0 0
- joint joint_6: origin xyz=0 0 0.1 rpy=0 0 0 -> xyz=0 0 0.05 rpy=0 0 0
